File: Motherboard/Projeto/Motherboard.kicad_sch (KiCad schematic)
At the start: 98 parts, among them J4 , J7 RJ14, J8 RJ14, M1a1 conn:CONN_01X25_LEFT, M1b1 conn:CONN_01X25_RIGHT, M2a1 conn:CONN_01X25_LEFT, M2b1 conn:CONN_01X25_RIGHT, M3a1 conn:CONN_01X25_LEFT, M3b1 conn:CONN_01X25_RIGHT, M4a1 conn:CONN_01X25_LEFT, M4b1 conn:CONN_01X25_RIGHT, M5a1 conn:CONN_01X25_LEFT, M5b1 conn:CONN_01X25_RIGHT, M6a1 conn:CONN_01X25_LEFT, M6b1 conn:CONN_01X25_RIGHT, M7a1 conn:CONN_01X25_LEFT, M7b1 conn:CONN_01X25_RIGHT, M8a1 conn:CONN_01X25_LEFT, M8b1 conn:CONN_01X25_RIGHT, M9a1 conn:CONN_01X09_LEFT, M9b1 conn:CONN_01X09_RIGHT, P1 CONN_02X08, P10 CONN_02X08, P11 CONN_02X08, P12 CONN_02X08, P13 CONN_02X08, P14 CONN_02X08, P15 CONN_02X08, P16 CONN_02X08, P2 CONN_02X08, P3 CONN_02X08, P4 CONN_02X08, P5 CONN_02X08, P6 CONN_02X08, P7 CONN_02X08, P8 CONN_02X08, P9 CONN_02X08, U1 CONN_02X12, U2 CONN_02X12, U3 CONN_02X12, U4 CONN_02X12

Commit message: RS485 inverted terminal updated on schematic
Connections:
- net A: now also J7.4 (T1); no longer J7.3 (R1)
- net B: now also J7.3 (R1); no longer J7.4 (T1)
Changed lines of the file:
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@@
     (effects (font (size 1.524 1.524)) (justify left bottom))
   )
-  (label "B" (at 377.19 195.58 180)
+  (label "A" (at 377.19 195.58 180)
     (effects (font (size 1.524 1.524)) (justify right bottom))
   )
@@
     (effects (font (size 1.524 1.524)) (justify left bottom))
   )
-  (label "A" (at 377.19 193.04 180)
+  (label "B" (at 377.19 193.04 180)
     (effects (font (size 1.524 1.524)) (justify right bottom))
   )
@@
       (reference "#PWR042") (unit 1) (value "GND") (footprint "")
     )
-    (path "/00000000-0000-0000-0000-0000576ab30b/00000000-0000-0000-0000-00005a69c007"
-      (reference "#PWR043") (unit 1) (value "+24V") (footprint "")
-    )
     (path "/00000000-0000-0000-0000-0000576ab30b/00000000-0000-0000-0000-00005a69c4a8"
-      (reference "#PWR044") (unit 1) (value "+24V") (footprint "")
+      (reference "#PWR044") (unit 1) (value "+12V") (footprint "")
     )
     (path "/00000000-0000-0000-0000-0000576ab30b/00000000-0000-0000-0000-00005a69c64d"
-      (reference "#PWR045") (unit 1) (value "+24V") (footprint "")
+      (reference "#PWR045") (unit 1) (value "+12V") (footprint "")
     )
     (path "/00000000-0000-0000-0000-0000576ab30b/00000000-0000-0000-0000-00005a69c70f"
-      (reference "#PWR046") (unit 1) (value "+24V") (footprint "")
+      (reference "#PWR046") (unit 1) (value "+12V") (footprint "")
     )
     (path "/00000000-0000-0000-0000-0000576ab30b/00000000-0000-0000-0000-00005a69c8a2"
-      (reference "#PWR047") (unit 1) (value "+24V") (footprint "")
+      (reference "#PWR047") (unit 1) (value "+12V") (footprint "")
     )
     (path "/00000000-0000-0000-0000-0000576ab30b/00000000-0000-0000-0000-00005a69c946"
-      (reference "#PWR048") (unit 1) (value "+24V") (footprint "")
+      (reference "#PWR048") (unit 1) (value "+12V") (footprint "")
     )
     (path "/00000000-0000-0000-0000-0000576ab30b/00000000-0000-0000-0000-00005a69ca6c"
-      (reference "#PWR049") (unit 1) (value "+24V") (footprint "")
+      (reference "#PWR049") (unit 1) (value "+12V") (footprint "")
     )
     (path "/00000000-0000-0000-0000-0000576ab30b/00000000-0000-0000-0000-00005a69ca82"
-      (reference "#PWR050") (unit 1) (value "+24V") (footprint "")
-    )
-    (path "/00000000-0000-0000-0000-0000576ab30b/00000000-0000-0000-0000-00005a70c8a9"
-      (reference "#PWR059") (unit 1) (value "+5V") (footprint "")
+      (reference "#PWR050") (unit 1) (value "+12V") (footprint "")
     )
     (path "/00000000-0000-0000-0000-0000576ab30b/00000000-0000-0000-0000-00005a70ca67"
@@
     )
     (path "/00000000-0000-0000-0000-0000576ab30b/00000000-0000-0000-0000-00005a8f09b2"
-      (reference "#PWR067") (unit 1) (value "+24V") (footprint "")
+      (reference "#PWR067") (unit 1) (value "+12V") (footprint "")
     )
     (path "/00000000-0000-0000-0000-0000576ab30b/00000000-0000-0000-0000-00005a8f0b5e"
@@
       (reference "#PWR?") (unit 1) (value "+5V") (footprint "")
     )
+    (path "/00000000-0000-0000-0000-0000576ab30b/4e4c13d8-0a01-49c9-a795-a1d30ff9efd2"
+      (reference "#PWR?") (unit 1) (value "+12V") (footprint "")
+    )
     (path "/00000000-0000-0000-0000-0000576ab30b/5493e8cd-8323-4518-b41a-1736b1fae7d0"
       (reference "#PWR?") (unit 1) (value "+5V") (footprint "")
     )
+    (path "/00000000-0000-0000-0000-0000576ab30b/577ae91e-cb35-46de-86b5-34d1ef80360a"
+      (reference "#PWR?") (unit 1) (value "+5V") (footprint "")
+    )
     (path "/00000000-0000-0000-0000-0000576ab30b/9292d21d-a1c5-4919-b2ca-d60a18782af4"
       (reference "#PWR?") (unit 1) (value "GND") (footprint "")
@@
     )
     (path "/00000000-0000-0000-0000-0000576ab30b/00000000-0000-0000-0000-000060d5e3d8"
-      (reference "P17") (unit 1) (value "SCREW_TERM_24V") (footprint "mods:OSTYK51102030")
+      (reference "P17") (unit 1) (value "SCREW_TERM_12V") (footprint "mods:OSTYK51102030")
     )
     (path "/00000000-0000-0000-0000-0000576ab30b/00000000-0000-0000-0000-000060db0b8b"
       (reference "P18") (unit 1) (value "SCREW_TERM_5V") (footprint "mods:OSTYK51102030")
     )
-    (path "/00000000-0000-0000-0000-0000576ab30b/00000000-0000-0000-0000-00005afb16b1"
+    (path "/00000000-0000-0000-0000-0000576ab30b/7f9cd99b-e372-41ec-91dd-ea62e68d3908"
       (reference "P38") (unit 1) (value "Jumper_Receptacle") (footprint "mods:Pin_Header_Straight_1x01_Pitch5.08mm")
     )
-    (path "/00000000-0000-0000-0000-0000576ab30b/00000000-0000-0000-0000-00005afb1e00"
+    (path "/00000000-0000-0000-0000-0000576ab30b/548b04a1-d840-46eb-8046-ea6d5b847536"
       (reference "P39") (unit 1) (value "Jumper_Receptacle") (footprint "mods:Pin_Header_Straight_1x01_Pitch5.08mm")
     )
-    (path "/00000000-0000-0000-0000-0000576ab30b/00000000-0000-0000-0000-00005afb1e95"
+    (path "/00000000-0000-0000-0000-0000576ab30b/eb530003-727b-4ecc-8b8f-441a3d94f9e6"
       (reference "P40") (unit 1) (value "Jumper_Receptacle") (footprint "mods:Pin_Header_Straight_1x01_Pitch5.08mm")
     )
